File: Electronics/FanController/_autosave-FanController.kicad_sch (KiCad schematic)
At the start: 5 parts, among them J1 POWER IN, J2 CONTROLLER IN/OUT, J3 PROGRAMMER, J4 SUPPLY SELECTOR, J5 FAN I/O

Commit message: Updated schematic
Connections:
- net +3.3V: no longer J2.1 (Pin_1), J3.1 (Pin_1)
- net +3.3VA: now also J3.1 (Pin_1)
- net VD: now also J2.1 (Pin_1)
- net VDD: now also J3.8 (Pin_8)
- no-connect marks 5 -> 4
Other:
- note added: "Target VCC"
- moved on the sheet: J2
