File: Electronics/FanController/FanController.kicad_sch (KiCad schematic)
At the start: 5 parts, among them J1 POWER IN, J2 CONTROLLER IN/OUT, J3 PROGRAMMER, J4 SUPPLY SELECTOR, J5 FAN I/O

Commit message: Started PCB-routing
Parts:
- J1: footprint (none) -> Connector_PinHeader_2.54mm:PinHeader_2x02_P2.54mm_Horizontal
- J2: footprint (none) -> Connector_PinHeader_2.54mm:PinHeader_2x04_P2.54mm_Horizontal
- J3: footprint (none) -> Connector_PinHeader_2.54mm:PinHeader_2x04_P2.54mm_Vertical
- J4: footprint (none) -> Connector_PinHeader_1.00mm:PinHeader_2x03_P1.00mm_Vertical
- J5: footprint (none) -> Connector_PinHeader_2.54mm:PinHeader_2x03_P2.54mm_Horizontal
Connections:
- net +3.3V: no longer J2.1 (Pin_1), J3.1 (Pin_1)
- net +3.3VA: now also J3.1 (Pin_1)
- net VD: now also J2.1 (Pin_1)
- net VDD: now also J3.8 (Pin_8)
- no-connect marks 5 -> 4
Other:
- note added: "Target VCC"
- moved on the sheet: J2

Commit message: Routed PCB-layout
Parts:
- J4: footprint Connector_PinHeader_1.00mm:PinHeader_2x03_P1.00mm_Vertical -> Connector_PinHeader_2.54mm:PinHeader_2x03_P2.54mm_Vertical
Connections:
- net +12V is gone; now on net +3.3V: J1.1 (Pin_1)
- net +12P: now also J1.3 (Pin_3)
- net +3.3V: no longer J1.3 (Pin_3)
- net +3.3VA: no longer J4.2 (Pin_2), J4.4 (Pin_4), J4.6 (Pin_6)
- net GND: now also J2.1 (Pin_1), J5.5 (Pin_5); no longer J2.7 (Pin_7), J5.3 (Pin_3)
- net Power_and_IO/OUT1: now also J5.3 (Pin_3); no longer J5.2 (Pin_2)
- net Power_and_IO/OUT2: now also J5.6 (Pin_6); no longer J5.4 (Pin_4)
- net Power_and_IO/PULSE_01_12V: now also J5.2 (Pin_2); no longer J5.5 (Pin_5)
- net Power_and_IO/PULSE_02_12V: now also J5.4 (Pin_4); no longer J5.6 (Pin_6)
- net VD: now also J2.7 (Pin_7); no longer J2.1 (Pin_1)
- net VDD: now also J3.2 (Pin_2); no longer J3.8 (Pin_8)
- net mcu/NRST: now also J3.8 (Pin_8); no longer J3.2 (Pin_2)
- new net +3.3VP: J4.2 (Pin_2), J4.4 (Pin_4), J4.6 (Pin_6)
